Commit message: used xacro for urdf

File: arm_description/urdf/arm.urdf.xacro (robot description, xacro)
@@ -1,4 +1,6 @@
-<?xml version="1.0"?>
-<robot name="arm">
+<?xml version="1.0" ?>
+<robot name="arm" xmlns:xacro="http://www.ros.org/wiki/xacro">
+  <!-- Add your robot description here, and include the gazebo macro -->
+  <xacro:include filename="$(find arm_description)/urdf/arm.gazebo.xacro" />
   <link name="base_link">
     <visual>
@@ -9,8 +11,8 @@
     </visual>
     <collision>
-      <geometry>
-        <mesh filename="package://arm_description/meshes/base_link.stl" scale="0.001 0.001 0.001"/>
-      </geometry>
-      <origin rpy="0 0 0" xyz="0 0 0"/>
+      <origin xyz="0 0 0.01" rpy="0 0 0"/> <!-- Adjust position and orientation as needed -->
+      <geometry>
+        <box size="0.1 0.1 0.08"/>
+      </geometry>
     </collision>
     <inertial>
@@ -32,8 +34,8 @@
     </visual>
     <collision>
-      <geometry>
-          <mesh filename="package://arm_description/meshes/base_turn.stl" scale="0.001 0.001 0.001"/>
-        </geometry>
-      <origin rpy="0 0 0" xyz="0 0 0"/>
+      <origin xyz="0 0.01 0" rpy="0 0 0"/> <!-- Adjust position and orientation as needed -->
+      <geometry>
+        <box size="0.06 0.08 0.01"/>
+      </geometry>
     </collision>
     <inertial>
@@ -56,8 +58,8 @@
     </visual>
     <collision>
-      <geometry>
-          <mesh filename="package://arm_description/meshes/base_turn_table_rot.stl" scale="0.001 0.001 0.001"/>
-        </geometry>
-      <origin rpy="0 0 0" xyz="0 0 0"/>
+      <origin xyz="0 0 0.003" rpy="0 0 0"/> <!-- Adjust position and orientation as needed -->
+      <geometry>
+        <box size="0.055 0.055 0.025"/>
+      </geometry>
     </collision>
     <inertial>
@@ -79,8 +81,8 @@
     </visual>
     <collision>
-      <geometry>
-          <mesh filename="package://arm_description/meshes/dyn.stl" scale="0.01 0.01 0.01"/>
-        </geometry>
-      <origin rpy="0 0 0" xyz="0 0 0"/>
+      <origin xyz="0.014 0 0" rpy="0 0 0"/> <!-- Adjust position and orientation as needed -->
+      <geometry>
+        <box size="0.051 0.031 0.041"/>
+      </geometry>
     </collision>
      <inertial>
@@ -114,8 +116,8 @@
     </visual>
     <collision>
-      <geometry>
-          <mesh filename="package://arm_description/meshes/f4_n_f3.stl" scale="0.001 0.001 0.001"/>
-        </geometry>
-      <origin rpy="0 0 0" xyz="0 0 0"/>
+      <origin xyz="-0.002 -0.01 0" rpy="0 0 0"/> <!-- Adjust position and orientation as needed -->
+      <geometry>
+        <box size="0.052 0.1 0.03"/>
+      </geometry>
     </collision>
      <inertial>
@@ -137,8 +139,8 @@
     </visual>
     <collision>
-      <geometry>
-          <mesh filename="package://arm_description/meshes/dyn.stl" scale="0.01 0.01 0.01"/>
-        </geometry>
-      <origin rpy="0 0 0" xyz="0 0 0"/>
+      <origin xyz="0.014 0 0" rpy="0 0 0"/> <!-- Adjust position and orientation as needed -->
+      <geometry>
+        <box size="0.051 0.031 0.041"/>
+      </geometry>
     </collision>
      <inertial>
@@ -172,8 +174,8 @@
     </visual>
     <collision>
-      <geometry>
-          <mesh filename="package://arm_description/meshes/f4_n_f3.stl" scale="0.001 0.001 0.001"/>
-        </geometry>
-      <origin rpy="0 0 0" xyz="0 0 0"/>
+      <origin xyz="-0.002 -0.01 0" rpy="0 0 0"/> <!-- Adjust position and orientation as needed -->
+      <geometry>
+        <box size="0.052 0.1 0.03"/>
+      </geometry>
     </collision>
     <inertial>
@@ -195,8 +197,8 @@
     </visual>
     <collision>
-      <geometry>
-          <mesh filename="package://arm_description/meshes/dyn.stl" scale="0.01 0.01 0.01"/>
-        </geometry>
-      <origin rpy="0 0 0" xyz="0 0 0"/>
+      <origin xyz="0.014 0 0" rpy="0 0 0"/> <!-- Adjust position and orientation as needed -->
+      <geometry>
+        <box size="0.051 0.031 0.041"/>
+      </geometry>
     </collision>
     <inertial>
@@ -230,8 +232,8 @@
     </visual>
     <collision>
-      <geometry>
-        <mesh filename="package://arm_description/meshes/wrist.stl" scale="0.001 0.001 0.001"/>
-      </geometry>
-      <origin rpy="0 0 0" xyz="0 0 0"/>
+      <origin xyz="0.003 0 -0.009" rpy="0 0 0"/> <!-- Adjust position and orientation as needed -->
+      <geometry>
+        <box size="0.055 0.06 0.044"/>
+      </geometry>
     </collision>
      <inertial>
@@ -252,10 +254,10 @@
       <origin rpy="0 0 0" xyz="0 0 0"/>
     </visual>
-    <collision>
-      <geometry>
-          <mesh filename="package://arm_description/meshes/dyn.stl" scale="0.01 0.01 0.01"/>
+      <collision>
+        <origin xyz="0.014 0 0" rpy="0 0 0"/> <!-- Adjust position and orientation as needed -->
+        <geometry>
+          <box size="0.051 0.031 0.041"/>
         </geometry>
-      <origin rpy="0 0 0" xyz="0 0 0"/>
-    </collision>
+      </collision>
     <inertial>
       <mass value="0.1"/>
@@ -288,8 +290,8 @@
     </visual>
     <collision>
-      <geometry>
-          <mesh filename="package://arm_description/meshes/the_crawer_base.stl" scale="0.001 0.001 0.001"/>
-        </geometry>
-      <origin rpy="0 0 0" xyz="0 0 0"/>
+      <origin xyz="0 0.005 0" rpy="0 0 0"/> <!-- Adjust position and orientation as needed -->
+      <geometry>
+        <box size="0.105 0.058 0.006"/>
+      </geometry>
     </collision>
     <inertial>
@@ -314,8 +316,8 @@
     </visual>
     <collision>
-      <geometry>
-          <mesh filename="package://arm_description/meshes/the_crawer.stl" scale="0.001 0.001 0.001"/>
-        </geometry>
-      <origin rpy="0 0 0" xyz="0 0 0"/>
+      <origin xyz="0.02 0 0.005" rpy="0 0 0"/> <!-- Adjust position and orientation as needed -->
+      <geometry>
+        <box size="0.07 0.04 0.045"/>
+      </geometry>
     </collision>
     <inertial>
@@ -340,52 +342,15 @@
     </visual>
     <collision>
-      <geometry>
-          <mesh filename="package://arm_description/meshes/the_crawer.stl" scale="0.001 0.001 0.001"/>
-        </geometry>
-      <origin rpy="0 0 0" xyz="0 0 0"/>
-    </collision>
-    <inertial>
-      <mass value="0.1"/>
-      <inertia ixx="6.90013881e+01" ixy="0.0" ixz="0.0" iyy="1.24554875e+02" iyz="0.0" izz="1.04295793e+02"/>
-    </inertial>
-  </link>
-  <gazebo reference="f4">
-    <material>Gazebo/Red</material>
-  </gazebo>
-  <gazebo reference="f5">
-    <material>Gazebo/Red</material>
-  </gazebo>
-  <gazebo reference="wrist">
-    <material>Gazebo/Red</material>
-  </gazebo>
-  <gazebo reference="crawer_base">
-    <material>Gazebo/Red</material>
-  </gazebo>
-  <gazebo reference="base_link">
-    <material>Gazebo/Red</material>
-  </gazebo>
-  <gazebo reference="base_turn">
-    <material>Gazebo/Red</material>
-  </gazebo>
-  <gazebo reference="base_turn_rot">
-    <material>Gazebo/Red</material>
-  </gazebo>
-  <gazebo reference="dyn2">
-    <material>Gazebo/Black</material>
-  </gazebo>
-  <gazebo reference="dyn3">
-    <material>Gazebo/Black</material>
-  </gazebo>
-  <gazebo reference="dyn4">
-    <material>Gazebo/Black</material>
-  </gazebo>
-  <gazebo reference="dyn5">
-    <material>Gazebo/Black</material>
-  </gazebo>
-  <gazebo reference="crawer_left">
-    <material>Gazebo/Red</material>
-  </gazebo>
-  <gazebo reference="crawer_right">
-    <material>Gazebo/Red</material>
-  </gazebo>
+      <origin xyz="0.02 0 0.005" rpy="0 0 0"/> <!-- Adjust position and orientation as needed -->
+      <geometry>
+        <box size="0.07 0.04 0.045"/>
+      </geometry>
+    </collision>
+    <inertial>
+      <mass value="0.1"/>
+      <inertia ixx="6.90013881e+01" ixy="0.0" ixz="0.0" iyy="1.24554875e+02" iyz="0.0" izz="1.04295793e+02"/>
+    </inertial>
+  </link>
+  <!-- This executes the xacro macro -->
+  <xacro:arm_gazebo/>
 </robot>

Commit message: added camera

File: arm_description/urdf/arm.urdf.xacro (robot description, xacro)
@@ -4,4 +4,5 @@
   <xacro:include filename="$(find arm_description)/urdf/arm.gazebo.xacro" />
   <xacro:include filename="$(find arm_description)/urdf/arm.transmission.xacro" />
+  <xacro:property name="camera_dim" value="0.025"/>
   <link name="base_link">
     <visual>
@@ -353,4 +354,31 @@
     </inertial>
   </link>
+  <!-- code added to add a camera -->
+  <joint name="camera_joint" type="fixed">
+    <axis xyz="0 1 0" />
+    <origin xyz="0 0 ${camera_dim}" rpy="0 0 0" />
+    <parent link="base_link" />
+    <child link="camera_link" />
+  </joint>
+  <link name="camera_link">
+    <collision>
+      <origin xyz="0 -0.04 -0.02" rpy="1.57 0 0" />
+      <geometry>
+        <box size="0.06 0.04 0.07" />
+      </geometry>
+    </collision>
+    <visual>
+      <origin xyz="0 -0.06 -0.02" rpy="1.57 0 0" />
+      <geometry>
+        <mesh filename="package://arm_description/meshes/camera.stl" scale="0.9 0.9 0.9"/>
+      </geometry>
+    </visual>
+    <inertial>
+      <mass value="1e-5" />
+      <origin xyz="0 0 0" rpy="0 0 0" />
+      <inertia ixx="1e-6" ixy="0" ixz="0" iyy="1e-6" iyz="0" izz="1e-6" />
+    </inertial>
+  </link>
+  <!-- end of camera link -->
   <!-- This executes the xacro macro -->
   <xacro:arm_gazebo/>
