Commit message: added camera.xacro

File: arm_description/urdf/arm.gazebo.xacro (robot description, xacro)
@@ -47,44 +47,4 @@
             <material>Gazebo/Red</material>
         </gazebo>
-        <!-- camera -->
-        <gazebo reference="camera_link">
-            <sensor type="camera" name="camera1">
-                <update_rate>30.0</update_rate>
-                <camera name="head">
-                    <horizontal_fov>1.3962634</horizontal_fov>
-                    <image>
-                        <width>800</width> <height>800</height> <format>
-                        R8G8B8</format>
-                    </image>
-                    <clip>
-                        <near>0.02</near> <far>300</far>
-                    </clip>
-                    <noise>
-                        <type>gaussian</type> <mean>0.0</mean> <stddev>0.007
-                    </stddev>
-                    </noise>
-                </camera>
-                <plugin name="camera_controller" filename="libgazebo_ros_camera.so"> ... </plugin>
-            </sensor>
-        </gazebo>
-        <!-- camera controller-->
-        <plugin name="camera_controller" filename="libgazebo_ros_camera.so">
-            <alwaysOn>true</alwaysOn>
-            <updateRate>0.0</updateRate>
-            <cameraName>camera</cameraName>
-            <imageTopicName>image_raw</imageTopicName>
-            <cameraInfoTopicName>camera_info</cameraInfoTopicName>
-            <frameName>camera_link_optical</frameName>
-            <hackBaseline>0.0</hackBaseline>
-            <distortionK1>0.0</distortionK1>
-            <distortionK2>0.0</distortionK2>
-            <distortionK3>0.0</distortionK3>
-            <distortionT1>0.0</distortionT1>
-            <distortionT2>0.0</distortionT2>
-            <CxPrime>0</CxPrime>
-            <Cx>0.0</Cx>
-            <Cy>0.0</Cy>
-            <focalLength>0.0</focalLength>
-        </plugin>
     </xacro:macro>
 </robot>

File: arm_description/urdf/arm.urdf.xacro (robot description, xacro)
@@ -4,5 +4,5 @@
   <xacro:include filename="$(find arm_description)/urdf/arm.gazebo.xacro" />
   <xacro:include filename="$(find arm_description)/urdf/arm.transmission.xacro" />
-  <xacro:property name="camera_dim" value="0.025"/>
+  <xacro:include filename="$(find arm_description)/urdf/camera.xacro" />
   <link name="base_link">
     <visual>
@@ -354,33 +354,7 @@
     </inertial>
   </link>
-  <!-- code added to add a camera -->
-  <joint name="camera_joint" type="fixed">
-    <axis xyz="0 1 0" />
-    <origin xyz="0 0 ${camera_dim}" rpy="0 0 0" />
-    <parent link="base_link" />
-    <child link="camera_link" />
-  </joint>
-  <link name="camera_link">
-    <collision>
-      <origin xyz="0 -0.04 -0.02" rpy="1.57 0 0" />
-      <geometry>
-        <box size="0.06 0.04 0.07" />
-      </geometry>
-    </collision>
-    <visual>
-      <origin xyz="0 -0.06 -0.02" rpy="1.57 0 0" />
-      <geometry>
-        <mesh filename="package://arm_description/meshes/camera.stl" scale="0.9 0.9 0.9"/>
-      </geometry>
-    </visual>
-    <inertial>
-      <mass value="1e-5" />
-      <origin xyz="0 0 0" rpy="0 0 0" />
-      <inertia ixx="1e-6" ixy="0" ixz="0" iyy="1e-6" iyz="0" izz="1e-6" />
-    </inertial>
-  </link>
-  <!-- end of camera link -->
   <!-- This executes the xacro macro -->
   <xacro:arm_gazebo/>
   <xacro:arm_transmission/>
+  <xacro:camera_sensor/>
 </robot>
