Commit message: Update camera.xacro

File: arm_description/urdf/camera.xacro (robot description, xacro)
@@ -5,5 +5,5 @@
         <joint name="camera_joint" type="fixed">
             <axis xyz="0 1 0" />
-            <origin xyz="0 0 0.025" rpy="0 0 0" />
+            <origin xyz="0.05 0 0.025" rpy="0 0 0" />
             <parent link="base_link" />
             <child link="camera_link" />
@@ -11,5 +11,5 @@
         <link name="camera_link">
             <collision>
-                <origin xyz="0.03 0 -0.02" rpy="1.57 0 1.57" />
+                <origin xyz="-0.02 0 -0.02" rpy="1.57 0 1.57" />
                 <geometry>
                     <box size="0.06 0.04 0.07" />
@@ -17,5 +17,5 @@
             </collision>
             <visual>
-                <origin xyz="0.05 0 -0.02" rpy="1.57 0 1.57" />
+                <origin xyz="0 0 -0.02" rpy="1.57 0 1.57" />
                 <geometry>
                     <mesh filename="package://arm_description/meshes/camera.stl" scale="0.9 0.9 0.9"/>
